File: Hardware/Prototype/tc0xC_proto.sch (EAGLE design)
At the start: 96 parts, among them IC1 AP2112M-3.3TRG1, Q1 2.5A/30V, Q2 MBT3904DW1T1, Q3 600mA/40V, Q4 MBT3904DW1T1, U2 ESP3212, U4 FT231XS, U5 W25Q32FVSS, Y1 26MHz, Y2 32.768kHz

Commit message: cleaned ripped up prototype
Parts:
- added C6: 4.7uF, SparkFun-Capacitors:0.1UF-0603-25V-(+80/-20%)
- added R20: 100, SparkFun-Resistors:10KOHM-0603-1/10W-1%
Connections:
- net 3.3V: now also C6.1, D33.VS, R20.1, R20.2
- net ACC_INT: now also D33.OUT
- net GND: now also C6.2, D33.GND
Other:
- moved on the sheet: C17
Changed lines of the file:
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@@
 <part name="R19" library="SparkFun-Resistors" deviceset="10KOHM" device="-0603-1/10W-1%" value="10k"/>
 <part name="SUPPLY3" library="SparkFun-Aesthetics" deviceset="3.3V" device=""/>
+<part name="R20" library="SparkFun-Resistors" deviceset="10KOHM" device="-0603-1/10W-1%" value="100"/>
+<part name="C6" library="SparkFun-Capacitors" deviceset="0.1UF" device="-0603-25V-(+80/-20%)" value="4.7uF"/>
 </parts>
 <sheets>
@@
 <attribute name="VALUE" x="-172.72" y="-25.4" size="1.778" layer="96" rot="MR0"/>
 </instance>
-<instance part="GND36" gate="1" x="-121.92" y="-22.86" smashed="yes" rot="MR0">
-<attribute name="VALUE" x="-119.38" y="-25.4" size="1.778" layer="96" rot="MR0"/>
+<instance part="GND36" gate="1" x="-137.16" y="0" smashed="yes" rot="MR0">
+<attribute name="VALUE" x="-134.62" y="-2.54" size="1.778" layer="96" rot="MR0"/>
 </instance>
 <instance part="U5" gate="G$1" x="-157.48" y="-10.16" smashed="yes">
@@
 <attribute name="VALUE" x="-170.18" y="-18.034" size="1.778" layer="96" align="top-left"/>
 </instance>
-<instance part="C17" gate="G$1" x="-121.92" y="-15.24" smashed="yes">
-<attribute name="NAME" x="-120.396" y="-12.319" size="1.778" layer="95" font="vector"/>
-<attribute name="VALUE" x="-120.396" y="-17.399" size="1.778" layer="96" font="vector"/>
+<instance part="C17" gate="G$1" x="-137.16" y="7.62" smashed="yes">
+<attribute name="NAME" x="-135.636" y="10.541" size="1.778" layer="95" font="vector"/>
+<attribute name="VALUE" x="-135.636" y="5.461" size="1.778" layer="96" font="vector"/>
 </instance>
 <instance part="R5" gate="G$1" x="-144.78" y="-45.72" smashed="yes" rot="R270">
@@
 <attribute name="NAME" x="-63.754" y="-54.864" size="1.27" layer="95" rot="R270"/>
 <attribute name="VALUE" x="-71.882" y="-54.864" size="1.27" layer="96" rot="R270"/>
+</instance>
+<instance part="R20" gate="G$1" x="-25.4" y="-53.34" smashed="yes">
+<attribute name="NAME" x="-25.4" y="-51.816" size="1.778" layer="95" font="vector" align="bottom-center"/>
+<attribute name="VALUE" x="-25.4" y="-54.864" size="1.778" layer="96" font="vector" align="top-center"/>
+</instance>
+<instance part="C6" gate="G$1" x="-30.48" y="-58.42" smashed="yes" rot="MR0">
+<attribute name="NAME" x="-32.004" y="-55.499" size="1.778" layer="95" font="vector" rot="MR0"/>
+<attribute name="VALUE" x="-32.004" y="-60.579" size="1.778" layer="96" font="vector" rot="MR0"/>
 </instance>
 </instances>
@@
 <segment>
 <pinref part="GND36" gate="1" pin="GND"/>
-<wire x1="-121.92" y1="-20.32" x2="-121.92" y2="-17.78" width="0.1524" layer="91"/>
+<wire x1="-137.16" y1="2.54" x2="-137.16" y2="5.08" width="0.1524" layer="91"/>
 <pinref part="C17" gate="G$1" pin="2"/>
 </segment>
@@
 <pinref part="R6" gate="G$1" pin="2"/>
 <pinref part="U$3" gate="G$1" pin="GND"/>
+</segment>
+<segment>
+<pinref part="D33" gate="G$1" pin="GND"/>
+<wire x1="-35.56" y1="-63.5" x2="-30.48" y2="-63.5" width="0.1524" layer="91"/>
+<pinref part="C6" gate="G$1" pin="2"/>
+<wire x1="-30.48" y1="-63.5" x2="-30.48" y2="-60.96" width="0.1524" layer="91"/>
+<junction x="-30.48" y="-63.5"/>
+<wire x1="-30.48" y1="-63.5" x2="-27.94" y2="-63.5" width="0.1524" layer="91"/>
+<label x="-27.94" y="-63.5" size="1.778" layer="95" xref="yes"/>
 </segment>
 </net>
@@
 <junction x="-139.7" y="-38.1"/>
 </segment>
+<segment>
+<pinref part="D33" gate="G$1" pin="VS"/>
+<wire x1="-35.56" y1="-53.34" x2="-30.48" y2="-53.34" width="0.1524" layer="91"/>
+<pinref part="R20" gate="G$1" pin="1"/>
+<junction x="-30.48" y="-53.34"/>
+<pinref part="C6" gate="G$1" pin="1"/>
+</segment>
+<segment>
+<pinref part="R20" gate="G$1" pin="2"/>
+<wire x1="-20.32" y1="-53.34" x2="-17.78" y2="-53.34" width="0.1524" layer="91"/>
+<wire x1="-15.24" y1="-53.34" x2="-17.78" y2="-53.34" width="0.1524" layer="91"/>
+<label x="-15.24" y="-53.34" size="1.778" layer="95" xref="yes"/>
+</segment>
 </net>
 <net name="SDA" class="0">
@@
 <pinref part="R9" gate="G$1" pin="2"/>
 <wire x1="-160.02" y1="-60.96" x2="-157.48" y2="-60.96" width="0.1524" layer="91"/>
-<label x="-160.02" y="-60.96" size="1.27" layer="95" rot="R180" xref="yes"/>
+<label x="-160.02" y="-60.96" size="1.778" layer="95" rot="R180" xref="yes"/>
 </segment>
 </net>
@@
 <segment>
 <pinref part="C17" gate="G$1" pin="1"/>
-<wire x1="-121.92" y1="-10.16" x2="-121.92" y2="-7.62" width="0.1524" layer="91"/>
-<wire x1="-119.38" y1="-7.62" x2="-121.92" y2="-7.62" width="0.1524" layer="91"/>
-<label x="-119.38" y="-7.62" size="1.27" layer="95" xref="yes"/>
+<wire x1="-137.16" y1="12.7" x2="-137.16" y2="15.24" width="0.1524" layer="91"/>
+<wire x1="-134.62" y1="15.24" x2="-137.16" y2="15.24" width="0.1524" layer="91"/>
+<label x="-134.62" y="15.24" size="1.27" layer="95" xref="yes"/>
 </segment>
 <segment>
@@
 <wire x1="-35.56" y1="12.7" x2="-38.1" y2="12.7" width="0.1524" layer="91"/>
 <label x="-35.56" y="12.7" size="1.27" layer="95" xref="yes"/>
+</segment>
+</net>
+<net name="ACC_INT" class="0">
+<segment>
+<pinref part="D33" gate="G$1" pin="OUT"/>
+<wire x1="-35.56" y1="-58.42" x2="-27.94" y2="-58.42" width="0.1524" layer="91"/>
+<label x="-27.94" y="-58.42" size="1.778" layer="95" xref="yes"/>
 </segment>
 </net>
@@
 </segment>
 </net>
-<net name="BUZZER_OUT" class="0">
-<segment>
-<pinref part="U2" gate="G$1" pin="(VSPICS0/HS1_DATA6)GPIO5"/>
-<wire x1="129.54" y1="63.5" x2="127" y2="63.5" width="0.1524" layer="91"/>
-<label x="129.54" y="63.5" size="1.27" layer="95" xref="yes"/>
-</segment>
-</net>
 <net name="T_B" class="0">
 <segment>
@@
 </segment>
 </net>
+<net name="BUZZER_OUT" class="0">
+<segment>
+<pinref part="U2" gate="G$1" pin="(VSPICS0/HS1_DATA6)GPIO5"/>
+<wire x1="127" y1="63.5" x2="129.54" y2="63.5" width="0.1524" layer="91"/>
+<label x="129.54" y="63.5" size="1.778" layer="95" xref="yes"/>
+</segment>
+</net>

Commit message: matrixed LEDs
Connections:
- new net N$21: D13.ANODE+, D14.ANODE+, D15.ANODE+, D16.ANODE+
- new net N$22: D17.ANODE+, D18.ANODE+, D19.ANODE+, D20.ANODE+
- new net N$6: D21.ANODE+, D22.ANODE+, D23.ANODE+, D24.ANODE+
- net CA1: now also D1.CATHODE-, D13.CATHODE-, D17.CATHODE-, D2.ANODE+, D21.CATHODE-, D3.ANODE+, D4.ANODE+, D5.CATHODE-, D9.CATHODE-
- net CA2: now also D1.ANODE+, D10.CATHODE-, D14.CATHODE-, D18.CATHODE-, D2.CATHODE-, D22.CATHODE-, D6.CATHODE-, D7.ANODE+, D8.ANODE+
- net CA3: now also D11.CATHODE-, D12.ANODE+, D15.CATHODE-, D19.CATHODE-, D23.CATHODE-, D3.CATHODE-, D5.ANODE+, D6.ANODE+, D7.CATHODE-
- net CA4: now also D10.ANODE+, D11.ANODE+, D12.CATHODE-, D16.CATHODE-, D20.CATHODE-, D24.CATHODE-, D4.CATHODE-, D8.CATHODE-, D9.ANODE+
Other:
- moved on the sheet: D1, D10, D11, D12, D13, D14, D15, D16, D17, D18, D19, D2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

Commit message: merged tKeepOut and drills
Parts:
- added R21, R22: 8.2, SparkFun-Resistors:10KOHM-0603-1/10W-1%
Connections:
- removed net N$21: D13.ANODE+, D14.ANODE+, D15.ANODE+, D16.ANODE+
- removed net N$22: D17.ANODE+, D18.ANODE+, D19.ANODE+, D20.ANODE+
- removed net T_START: U2.(ADC2:0/TOUCH0/RTC10/SPIHD)GPIO4
- new net IR_OUT: R21.1, R22.1, U2.(ADC2:0/TOUCH0/RTC10/SPIHD)GPIO4
- new net N$5: D27.A, R21.2
- net CA5: now also D13.ANODE+, D14.ANODE+, D15.ANODE+, D16.ANODE+
- net CA6: now also D17.ANODE+, D18.ANODE+, D19.ANODE+, D20.ANODE+
- net CA7: now also D21.ANODE+, D22.ANODE+, D23.ANODE+, D24.ANODE+
- net GND: now also D27.C, D28.C
- net N$6: now also D28.A, R22.2; no longer D21.ANODE+, D22.ANODE+, D23.ANODE+, D24.ANODE+
Changed lines of the file:
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@@
 <layer number="2" name="Route2" color="1" fill="3" visible="no" active="no"/>
 <layer number="3" name="Route3" color="4" fill="3" visible="no" active="no"/>
+<layer number="4" name="Route4" color="1" fill="4" visible="no" active="no"/>
+<layer number="5" name="Route5" color="4" fill="4" visible="no" active="no"/>
+<layer number="6" name="Route6" color="1" fill="8" visible="no" active="no"/>
+<layer number="7" name="Route7" color="4" fill="8" visible="no" active="no"/>
+<layer number="8" name="Route8" color="1" fill="2" visible="no" active="no"/>
+<layer number="9" name="Route9" color="4" fill="2" visible="no" active="no"/>
+<layer number="10" name="Route10" color="1" fill="7" visible="no" active="no"/>
+<layer number="11" name="Route11" color="4" fill="7" visible="no" active="no"/>
+<layer number="12" name="Route12" color="1" fill="5" visible="no" active="no"/>
+<layer number="13" name="Route13" color="4" fill="5" visible="no" active="no"/>
 <layer number="14" name="Route14" color="1" fill="6" visible="no" active="no"/>
 <layer number="15" name="Route15" color="4" fill="6" visible="no" active="no"/>
@@
 <part name="R20" library="SparkFun-Resistors" deviceset="10KOHM" device="-0603-1/10W-1%" value="100"/>
 <part name="C6" library="SparkFun-Capacitors" deviceset="0.1UF" device="-0603-25V-(+80/-20%)" value="4.7uF"/>
+<part name="GND11" library="supply1" library_urn="urn:adsk.eagle:library:371" deviceset="GND" device=""/>
+<part name="GND17" library="supply1" library_urn="urn:adsk.eagle:library:371" deviceset="GND" device=""/>
+<part name="R21" library="SparkFun-Resistors" deviceset="10KOHM" device="-0603-1/10W-1%" value="8.2"/>
+<part name="R22" library="SparkFun-Resistors" deviceset="10KOHM" device="-0603-1/10W-1%" value="8.2"/>
 </parts>
 <sheets>
@@
 <attribute name="VALUE" x="-32.004" y="-60.579" size="1.778" layer="96" font="vector" rot="MR0"/>
 </instance>
+<instance part="GND11" gate="1" x="-81.28" y="-66.04" smashed="yes">
+<attribute name="VALUE" x="-83.82" y="-68.58" size="1.778" layer="96"/>
+</instance>
+<instance part="GND17" gate="1" x="-68.58" y="-66.04" smashed="yes">
+<attribute name="VALUE" x="-71.12" y="-68.58" size="1.778" layer="96"/>
+</instance>
+<instance part="R21" gate="G$1" x="-81.28" y="-45.72" smashed="yes" rot="R270">
+<attribute name="NAME" x="-79.756" y="-45.72" size="1.778" layer="95" font="vector" rot="R270" align="bottom-center"/>
+<attribute name="VALUE" x="-82.804" y="-45.72" size="1.778" layer="96" font="vector" rot="R270" align="top-center"/>
+</instance>
+<instance part="R22" gate="G$1" x="-68.58" y="-45.72" smashed="yes" rot="R270">
+<attribute name="NAME" x="-67.056" y="-45.72" size="1.778" layer="95" font="vector" rot="R270" align="bottom-center"/>
+<attribute name="VALUE" x="-70.104" y="-45.72" size="1.778" layer="96" font="vector" rot="R270" align="top-center"/>
+</instance>
 </instances>
 <busses>
@@
 <wire x1="-30.48" y1="-63.5" x2="-27.94" y2="-63.5" width="0.1524" layer="91"/>
 <label x="-27.94" y="-63.5" size="1.778" layer="95" xref="yes"/>
+</segment>
+<segment>
+<pinref part="D27" gate="G$1" pin="C"/>
+<pinref part="GND11" gate="1" pin="GND"/>
+</segment>
+<segment>
+<pinref part="D28" gate="G$1" pin="C"/>
+<pinref part="GND17" gate="1" pin="GND"/>
 </segment>
 </net>
@@
 <label x="-35.56" y="17.78" size="1.27" layer="95" xref="yes"/>
 </segment>
+<segment>
+<pinref part="D16" gate="G$1" pin="ANODE+"/>
+<pinref part="D13" gate="G$1" pin="ANODE+"/>
+<wire x1="63.5" y1="22.86" x2="71.12" y2="22.86" width="0.1524" layer="91"/>
+<wire x1="71.12" y1="22.86" x2="71.12" y2="10.16" width="0.1524" layer="91"/>
+<pinref part="D14" gate="G$1" pin="ANODE+"/>
+<wire x1="71.12" y1="10.16" x2="71.12" y2="-2.54" width="0.1524" layer="91"/>
+<wire x1="71.12" y1="-2.54" x2="71.12" y2="-7.62" width="0.1524" layer="91"/>
+<wire x1="63.5" y1="10.16" x2="71.12" y2="10.16" width="0.1524" layer="91"/>
+<junction x="71.12" y="10.16"/>
+<pinref part="D15" gate="G$1" pin="ANODE+"/>
+<wire x1="63.5" y1="-2.54" x2="71.12" y2="-2.54" width="0.1524" layer="91"/>
+<junction x="71.12" y="-2.54"/>
+<wire x1="71.12" y1="-27.94" x2="71.12" y2="-2.54" width="0.1524" layer="91"/>
+<wire x1="-5.08" y1="-27.94" x2="63.5" y2="-27.94" width="0.1524" layer="91"/>
+<wire x1="63.5" y1="-27.94" x2="71.12" y2="-27.94" width="0.1524" layer="91"/>
+<wire x1="63.5" y1="-17.78" x2="63.5" y2="-27.94" width="0.1524" layer="91"/>
+<junction x="63.5" y="-27.94"/>
+<label x="-5.08" y="-27.94" size="1.778" layer="95" rot="R180" xref="yes"/>
+</segment>
 </net>
 <net name="CA6" class="0">
@@
 <label x="-35.56" y="15.24" size="1.27" layer="95" xref="yes"/>
 </segment>
+<segment>
+<pinref part="D17" gate="G$1" pin="ANODE+"/>
+<wire x1="81.28" y1="22.86" x2="88.9" y2="22.86" width="0.1524" layer="91"/>
+<wire x1="88.9" y1="22.86" x2="88.9" y2="10.16" width="0.1524" layer="91"/>
+<pinref part="D18" gate="G$1" pin="ANODE+"/>
+<wire x1="88.9" y1="10.16" x2="88.9" y2="-2.54" width="0.1524" layer="91"/>
+<wire x1="81.28" y1="10.16" x2="88.9" y2="10.16" width="0.1524" layer="91"/>
+<junction x="88.9" y="10.16"/>
+<pinref part="D19" gate="G$1" pin="ANODE+"/>
+<wire x1="81.28" y1="-2.54" x2="88.9" y2="-2.54" width="0.1524" layer="91"/>
+<junction x="88.9" y="-2.54"/>
+<wire x1="88.9" y1="-35.56" x2="88.9" y2="-2.54" width="0.1524" layer="91"/>
+<wire x1="88.9" y1="-35.56" x2="81.28" y2="-35.56" width="0.1524" layer="91"/>
+<label x="-5.08" y="-35.56" size="1.778" layer="95" rot="R180" xref="yes"/>
+<pinref part="D20" gate="G$1" pin="ANODE+"/>
+<wire x1="81.28" y1="-35.56" x2="-5.08" y2="-35.56" width="0.1524" layer="91"/>
+<wire x1="81.28" y1="-17.78" x2="81.28" y2="-35.56" width="0.1524" layer="91"/>
+<junction x="81.28" y="-35.56"/>
+</segment>
 </net>
 <net name="CA7" class="0">
@@
 <label x="-35.56" y="12.7" size="1.27" layer="95" xref="yes"/>
 </segment>
-</net>
-<net name="ACC_INT" class="0">
-<segment>
-<pinref part="D33" gate="G$1" pin="OUT"/>
-<wire x1="-35.56" y1="-58.42" x2="-27.94" y2="-58.42" width="0.1524" layer="91"/>
-<label x="-27.94" y="-58.42" size="1.778" layer="95" xref="yes"/>
-</segment>
-</net>
-<net name="N$6" class="0">
 <segment>
 <pinref part="D21" gate="G$1" pin="ANODE+"/>
@@
 <wire x1="96.52" y1="-17.78" x2="96.52" y2="-22.86" width="0.1524" layer="91"/>
 <wire x1="96.52" y1="-22.86" x2="101.6" y2="-22.86" width="0.1524" layer="91"/>
-</segment>
-</net>
-<net name="N$21" class="0">
-<segment>
-<pinref part="D13" gate="G$1" pin="ANODE+"/>
-<wire x1="63.5" y1="22.86" x2="71.12" y2="22.86" width="0.1524" layer="91"/>
-<wire x1="71.12" y1="22.86" x2="71.12" y2="10.16" width="0.1524" layer="91"/>
-<pinref part="D14" gate="G$1" pin="ANODE+"/>
-<wire x1="71.12" y1="10.16" x2="71.12" y2="-2.54" width="0.1524" layer="91"/>
-<wire x1="71.12" y1="-2.54" x2="71.12" y2="-7.62" width="0.1524" layer="91"/>
-<wire x1="63.5" y1="10.16" x2="71.12" y2="10.16" width="0.1524" layer="91"/>
-<junction x="71.12" y="10.16"/>
-<pinref part="D15" gate="G$1" pin="ANODE+"/>
-<wire x1="63.5" y1="-2.54" x2="71.12" y2="-2.54" width="0.1524" layer="91"/>
-<junction x="71.12" y="-2.54"/>
-<pinref part="D16" gate="G$1" pin="ANODE+"/>
-<wire x1="63.5" y1="-17.78" x2="63.5" y2="-22.86" width="0.1524" layer="91"/>
-<wire x1="63.5" y1="-22.86" x2="71.12" y2="-22.86" width="0.1524" layer="91"/>
-<wire x1="71.12" y1="-22.86" x2="71.12" y2="-2.54" width="0.1524" layer="91"/>
-</segment>
-</net>
-<net name="N$22" class="0">
-<segment>
-<pinref part="D17" gate="G$1" pin="ANODE+"/>
-<wire x1="81.28" y1="22.86" x2="88.9" y2="22.86" width="0.1524" layer="91"/>
-<wire x1="88.9" y1="22.86" x2="88.9" y2="10.16" width="0.1524" layer="91"/>
-<pinref part="D18" gate="G$1" pin="ANODE+"/>
-<wire x1="88.9" y1="10.16" x2="88.9" y2="-2.54" width="0.1524" layer="91"/>
-<wire x1="81.28" y1="10.16" x2="88.9" y2="10.16" width="0.1524" layer="91"/>
-<junction x="88.9" y="10.16"/>
-<pinref part="D19" gate="G$1" pin="ANODE+"/>
-<wire x1="81.28" y1="-2.54" x2="88.9" y2="-2.54" width="0.1524" layer="91"/>
-<junction x="88.9" y="-2.54"/>
-<pinref part="D20" gate="G$1" pin="ANODE+"/>
-<wire x1="81.28" y1="-17.78" x2="81.28" y2="-22.86" width="0.1524" layer="91"/>
-<wire x1="81.28" y1="-22.86" x2="88.9" y2="-22.86" width="0.1524" layer="91"/>
-<wire x1="88.9" y1="-22.86" x2="88.9" y2="-2.54" width="0.1524" layer="91"/>
+<wire x1="101.6" y1="-22.86" x2="101.6" y2="-43.18" width="0.1524" layer="91"/>
+<junction x="101.6" y="-22.86"/>
+<wire x1="101.6" y1="-43.18" x2="-5.08" y2="-43.18" width="0.1524" layer="91"/>
+<label x="-5.08" y="-43.18" size="1.778" layer="95" rot="R180" xref="yes"/>
+</segment>
+</net>
+<net name="ACC_INT" class="0">
+<segment>
+<pinref part="D33" gate="G$1" pin="OUT"/>
+<wire x1="-35.56" y1="-58.42" x2="-27.94" y2="-58.42" width="0.1524" layer="91"/>
+<label x="-27.94" y="-58.42" size="1.778" layer="95" xref="yes"/>
+</segment>
+</net>
+<net name="N$5" class="0">
+<segment>
+<pinref part="D27" gate="G$1" pin="A"/>
+<pinref part="R21" gate="G$1" pin="2"/>
+</segment>
+</net>
+<net name="N$6" class="0">
+<segment>
+<pinref part="D28" gate="G$1" pin="A"/>
+<pinref part="R22" gate="G$1" pin="2"/>
+</segment>
+</net>
+<net name="IR_OUT" class="0">
+<segment>
+<pinref part="R21" gate="G$1" pin="1"/>
+<wire x1="-81.28" y1="-40.64" x2="-81.28" y2="-38.1" width="0.1524" layer="91"/>
+<label x="-81.28" y="-38.1" size="1.778" layer="95" rot="R180" xref="yes"/>
+</segment>
+<segment>
+<pinref part="R22" gate="G$1" pin="1"/>
+<wire x1="-68.58" y1="-40.64" x2="-68.58" y2="-33.02" width="0.1524" layer="91"/>
+<label x="-68.58" y="-33.02" size="1.778" layer="95" rot="R180" xref="yes"/>
 </segment>
 </net>
@@
 </segment>
 </net>
-<net name="T_START" class="0">
+<net name="IR_OUT" class="0">
 <segment>
 <pinref part="U2" gate="G$1" pin="(ADC2:0/TOUCH0/RTC10/SPIHD)GPIO4"/>

Commit message: right angle momentary placement
Parts:
- added S3: TL3340AF160QG, TL3340AF160QG:TL3340AF160QG
Changed lines of the file:
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@@
 <part name="R21" library="SparkFun-Resistors" deviceset="10KOHM" device="-0603-1/10W-1%" value="8.2"/>
 <part name="R22" library="SparkFun-Resistors" deviceset="10KOHM" device="-0603-1/10W-1%" value="8.2"/>
+<part name="S3" library="TL3340AF160QG" deviceset="TL3340AF160QG" device=""/>
 </parts>
 <sheets>
@@
 <attribute name="VALUE" x="179.324" y="-39.624" size="1.778" layer="96"/>
 </instance>
+<instance part="S3" gate="G$1" x="-93.98" y="25.4" smashed="yes">
+<attribute name="NAME" x="-96.52" y="27.94" size="1.27" layer="95"/>
+<attribute name="VALUE" x="-96.52" y="22.86" size="1.27" layer="96" align="top-left"/>
+</instance>
 </instances>
