File: Hardware/Prototype/tc0xC_proto.sch (EAGLE design)
At the start: 101 parts, among them IC1 AP2112M-3.3TRG1, Q1 2.5A/30V, Q2 MBT3904DW1T1, Q3 600mA/40V, Q4 MBT3904DW1T1, U2 ESP3212, U4 FT231XS, U5 W25Q32FVSS, Y1 26MHz, Y2 32.768kHz

Commit message: routed
Parts:
- removed S1: PTS526, IDEO-Switches:PTS526
Connections:
- removed net CA8: U1.CA8
- removed net CA9: U1.CA9
- removed net RX_IN: U2.(HS1_DATA5)GPIO17
- removed net TX_IN: U2.(HS1_DATA4)GPIO16
- removed net XMARK: U2.(VSPIQ/HS2_DATA2)GPIO19
- net CHIP_PU: now also S3.NO; no longer S1.P$2
- net GND: now also S3.COM_1, S3.COM_2; no longer S1.P$1
Other:
- moved on the sheet: S3
Changed lines of the file:
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@@
 <part name="GND16" library="SparkFun-Aesthetics" deviceset="GND" device=""/>
 <part name="SUPPLY23" library="SparkFun-Aesthetics" deviceset="3.3V" device=""/>
-<part name="S1" library="IDEO-Switches" deviceset="PTS526" device=""/>
 <part name="S2" library="IDEO-Switches" deviceset="CUS-12B" device=""/>
 <part name="SUPPLY15" library="SparkFun-Aesthetics" deviceset="V_BATT" device=""/>
@@
 </segment>
 <segment>
+<pinref part="R20" gate="G$1" pin="1"/>
+<pinref part="C6" gate="G$1" pin="1"/>
 <pinref part="D33" gate="G$1" pin="VS"/>
 <wire x1="-35.56" y1="-53.34" x2="-30.48" y2="-53.34" width="0.1524" layer="91"/>
-<pinref part="R20" gate="G$1" pin="1"/>
 <junction x="-30.48" y="-53.34"/>
-<pinref part="C6" gate="G$1" pin="1"/>
 </segment>
 <segment>
@@
 </segment>
 </net>
-<net name="FLASH_SDO" class="0">
-<segment>
-<wire x1="-172.72" y1="-10.16" x2="-175.26" y2="-10.16" width="0.1524" layer="91"/>
-<label x="-175.26" y="-10.16" size="1.27" layer="95" rot="R180" xref="yes"/>
-<pinref part="U5" gate="G$1" pin="SO(D1)"/>
-</segment>
-</net>
 <net name="FLASH_SCK" class="0">
 <segment>
@@
 <label x="-139.7" y="-12.7" size="1.27" layer="95" xref="yes"/>
 <pinref part="U5" gate="G$1" pin="SCK"/>
-</segment>
-</net>
-<net name="FLASH_SCS" class="0">
-<segment>
-<wire x1="-172.72" y1="-7.62" x2="-175.26" y2="-7.62" width="0.1524" layer="91"/>
-<label x="-175.26" y="-7.62" size="1.27" layer="95" rot="R180" xref="yes"/>
-<pinref part="U5" gate="G$1" pin="!CS!"/>
 </segment>
 </net>
@@
 </segment>
 </net>
-<net name="CA8" class="0">
-<segment>
-<pinref part="U1" gate="G$1" pin="CA8"/>
-<wire x1="-35.56" y1="10.16" x2="-38.1" y2="10.16" width="0.1524" layer="91"/>
-<label x="-35.56" y="10.16" size="1.27" layer="95" xref="yes"/>
-</segment>
-</net>
-<net name="CA9" class="0">
-<segment>
-<pinref part="U1" gate="G$1" pin="CA9"/>
-<wire x1="-35.56" y1="7.62" x2="-38.1" y2="7.62" width="0.1524" layer="91"/>
-<label x="-35.56" y="7.62" size="1.27" layer="95" xref="yes"/>
-</segment>
-</net>
 <net name="CA4" class="0">
 <segment>
@@
 <wire x1="-68.58" y1="-40.64" x2="-68.58" y2="-33.02" width="0.1524" layer="91"/>
 <label x="-68.58" y="-33.02" size="1.778" layer="95" rot="R180" xref="yes"/>
+</segment>
+</net>
+<net name="FLASH_SCS" class="0">
+<segment>
+<pinref part="U5" gate="G$1" pin="!CS!"/>
+<wire x1="-172.72" y1="-7.62" x2="-175.26" y2="-7.62" width="0.1524" layer="91"/>
+<label x="-175.26" y="-7.62" size="1.27" layer="95" rot="R180" xref="yes"/>
+</segment>
+</net>
+<net name="FLASH_SDO" class="0">
+<segment>
+<pinref part="U5" gate="G$1" pin="SO(D1)"/>
+<wire x1="-172.72" y1="-10.16" x2="-175.26" y2="-10.16" width="0.1524" layer="91"/>
+<label x="-175.26" y="-10.16" size="1.27" layer="95" rot="R180" xref="yes"/>
 </segment>
 </net>
@@
 <attribute name="VALUE" x="-48.26" y="3.81" size="1.778" layer="96" font="vector" rot="R180" align="center-left"/>
 </instance>
-<instance part="GND1" gate="1" x="-109.22" y="33.02" smashed="yes">
-<attribute name="VALUE" x="-111.76" y="30.48" size="1.778" layer="96"/>
+<instance part="GND1" gate="1" x="-119.38" y="33.02" smashed="yes">
+<attribute name="VALUE" x="-119.38" y="30.48" size="1.778" layer="96"/>
 </instance>
 <instance part="R1" gate="G$1" x="-93.98" y="45.72" smashed="yes" rot="R90">
@@
 <attribute name="VALUE" x="-69.596" y="21.336" size="1.778" layer="96"/>
 </instance>
-<instance part="S1" gate="G$1" x="-101.6" y="38.1" smashed="yes">
-<attribute name="NAME" x="-104.14" y="41.656" size="1.524" layer="95"/>
-</instance>
 <instance part="S2" gate="G$1" x="193.04" y="-30.48" smashed="yes" rot="R90">
 <attribute name="NAME" x="187.452" y="-33.02" size="1.6764" layer="95" font="vector" ratio="10" rot="R90"/>
@@
 <attribute name="VALUE" x="179.324" y="-39.624" size="1.778" layer="96"/>
 </instance>
-<instance part="S3" gate="G$1" x="-93.98" y="25.4" smashed="yes">
-<attribute name="NAME" x="-96.52" y="27.94" size="1.27" layer="95"/>
-<attribute name="VALUE" x="-96.52" y="22.86" size="1.27" layer="96" align="top-left"/>
+<instance part="S3" gate="G$1" x="-104.14" y="38.1" smashed="yes">
+<attribute name="NAME" x="-106.68" y="40.64" size="1.27" layer="95"/>
+<attribute name="VALUE" x="-106.68" y="35.56" size="1.27" layer="96" align="top-left"/>
 </instance>
 </instances>
@@
 </segment>
 <segment>
-<wire x1="-106.68" y1="38.1" x2="-109.22" y2="38.1" width="0.1524" layer="91"/>
-<wire x1="-109.22" y1="38.1" x2="-109.22" y2="35.56" width="0.1524" layer="91"/>
+<wire x1="-119.38" y1="38.1" x2="-119.38" y2="35.56" width="0.1524" layer="91"/>
 <pinref part="GND1" gate="1" pin="GND"/>
-<pinref part="S1" gate="G$1" pin="P$1"/>
+<pinref part="S3" gate="G$1" pin="COM_1"/>
+<wire x1="-119.38" y1="38.1" x2="-114.3" y2="38.1" width="0.1524" layer="91"/>
+<wire x1="-114.3" y1="38.1" x2="-114.3" y2="40.64" width="0.1524" layer="91"/>
+<pinref part="S3" gate="G$1" pin="COM_2"/>
+<wire x1="-114.3" y1="38.1" x2="-114.3" y2="35.56" width="0.1524" layer="91"/>
+<junction x="-114.3" y="38.1"/>
 </segment>
 <segment>
@@
 <wire x1="-93.98" y1="40.64" x2="-93.98" y2="38.1" width="0.1524" layer="91"/>
 <junction x="-93.98" y="38.1"/>
-<pinref part="S1" gate="G$1" pin="P$2"/>
+<pinref part="S3" gate="G$1" pin="NO"/>
 </segment>
 </net>
@@
 </segment>
 </net>
-<net name="TX_IN" class="0">
-<segment>
-<pinref part="U2" gate="G$1" pin="(HS1_DATA4)GPIO16"/>
-<wire x1="127" y1="60.96" x2="129.54" y2="60.96" width="0.1524" layer="91"/>
-<label x="129.54" y="60.96" size="1.27" layer="95" xref="yes"/>
-</segment>
-</net>
-<net name="RX_IN" class="0">
-<segment>
-<pinref part="U2" gate="G$1" pin="(HS1_DATA5)GPIO17"/>
-<wire x1="127" y1="58.42" x2="129.54" y2="58.42" width="0.1524" layer="91"/>
-<label x="129.54" y="58.42" size="1.27" layer="95" xref="yes"/>
-</segment>
-</net>
-<net name="XMARK" class="0">
-<segment>
-<pinref part="U2" gate="G$1" pin="(VSPIQ/HS2_DATA2)GPIO19"/>
-<wire x1="129.54" y1="53.34" x2="127" y2="53.34" width="0.1524" layer="91"/>
-</segment>
-</net>

Commit message: routed
Parts:
- added TP2, TP3: TPSTP08R, testpad:TPSTP08R
- C6: value 4.7uF -> 0.1uF; device SparkFun-Capacitors:0.1UF-0603-25V-(+80/-20%) -> SparkFun-Capacitors:10PF-0603-50V-5%
Connections:
- removed net T_B: Q4Q2.C, U2.(ADC2:1/TOUCH1/RTC11/CLK_OUT1)GPIO0
- new net T_B1: TP2.PP, U2.(ADC2:1/TOUCH1/RTC11/CLK_OUT1)GPIO0
- new net T_B2: Q4Q2.C, TP3.PP
- net 3.3V: now also C6.2; no longer C6.1
- net GND: now also C6.1; no longer C6.2
Other:
- moved on the sheet: C6
Changed lines of the file:
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@@
 <?xml version="1.0" encoding="utf-8"?>
 <!DOCTYPE eagle SYSTEM "eagle.dtd">
-<eagle version="9.6.1">
+<eagle version="9.6.2">
 <drawing>
 <settings>
@@
 <part name="SUPPLY3" library="SparkFun-Aesthetics" deviceset="3.3V" device=""/>
 <part name="R20" library="SparkFun-Resistors" deviceset="10KOHM" device="-0603-1/10W-1%" value="100"/>
-<part name="C6" library="SparkFun-Capacitors" deviceset="0.1UF" device="-0603-25V-(+80/-20%)" value="4.7uF"/>
 <part name="GND11" library="supply1" library_urn="urn:adsk.eagle:library:371" deviceset="GND" device=""/>
 <part name="GND17" library="supply1" library_urn="urn:adsk.eagle:library:371" deviceset="GND" device=""/>
@@
 <part name="R22" library="SparkFun-Resistors" deviceset="10KOHM" device="-0603-1/10W-1%" value="8.2"/>
 <part name="S3" library="TL3340AF160QG" deviceset="TL3340AF160QG" device=""/>
+<part name="TP2" library="testpad" library_urn="urn:adsk.eagle:library:385" deviceset="TPS" device="TP08R" package3d_urn="urn:adsk.eagle:package:27956/1"/>
+<part name="TP3" library="testpad" library_urn="urn:adsk.eagle:library:385" deviceset="TPS" device="TP08R" package3d_urn="urn:adsk.eagle:package:27956/1"/>
+<part name="GND37" library="supply1" library_urn="urn:adsk.eagle:library:371" deviceset="GND" device=""/>
+<part name="C6" library="SparkFun-Capacitors" deviceset="10PF" device="-0603-50V-5%" value="0.1uF"/>
+<part name="GND41" library="supply1" library_urn="urn:adsk.eagle:library:371" deviceset="GND" device=""/>
 </parts>
 <sheets>
@@
 <text x="-157.48" y="-50.8" size="2.54" layer="94" align="bottom-center">BUZZER</text>
 <text x="-55.88" y="43.18" size="2.54" layer="94" align="bottom-center">LED Driver</text>
-<text x="-55.88" y="-40.64" size="2.54" layer="94" align="bottom-center">Infrared</text>
+<text x="-45.72" y="-45.72" size="2.54" layer="94" align="bottom-center">Infrared</text>
 </plain>
 <instances>
@@
 <attribute name="VALUE" x="-25.4" y="-54.864" size="1.778" layer="96" font="vector" align="top-center"/>
 </instance>
-<instance part="C6" gate="G$1" x="-30.48" y="-58.42" smashed="yes" rot="MR0">
-<attribute name="NAME" x="-32.004" y="-55.499" size="1.778" layer="95" font="vector" rot="MR0"/>
-<attribute name="VALUE" x="-32.004" y="-60.579" size="1.778" layer="96" font="vector" rot="MR0"/>
-</instance>
 <instance part="GND11" gate="1" x="-81.28" y="-66.04" smashed="yes">
 <attribute name="VALUE" x="-83.82" y="-68.58" size="1.778" layer="96"/>
@@
 <attribute name="NAME" x="-67.056" y="-45.72" size="1.778" layer="95" font="vector" rot="R270" align="bottom-center"/>
 <attribute name="VALUE" x="-70.104" y="-45.72" size="1.778" layer="96" font="vector" rot="R270" align="top-center"/>
+</instance>
+<instance part="GND37" gate="1" x="-27.94" y="-66.04" smashed="yes">
+<attribute name="VALUE" x="-30.48" y="-68.58" size="1.778" layer="96"/>
+</instance>
+<instance part="C6" gate="G$1" x="-30.48" y="-48.26" smashed="yes">
+<attribute name="NAME" x="-29.718" y="-43.942" size="1.778" layer="95" font="vector" rot="MR180"/>
+<attribute name="VALUE" x="-33.02" y="-50.546" size="1.778" layer="96" font="vector"/>
+</instance>
+<instance part="GND41" gate="1" x="-30.48" y="-40.64" smashed="yes" rot="R180">
+<attribute name="VALUE" x="-27.94" y="-38.1" size="1.778" layer="96" rot="R180"/>
 </instance>
 </instances>
@@
 </segment>
 <segment>
-<pinref part="D33" gate="G$1" pin="GND"/>
-<wire x1="-35.56" y1="-63.5" x2="-30.48" y2="-63.5" width="0.1524" layer="91"/>
-<pinref part="C6" gate="G$1" pin="2"/>
-<wire x1="-30.48" y1="-63.5" x2="-30.48" y2="-60.96" width="0.1524" layer="91"/>
-<junction x="-30.48" y="-63.5"/>
-<wire x1="-30.48" y1="-63.5" x2="-27.94" y2="-63.5" width="0.1524" layer="91"/>
-<label x="-27.94" y="-63.5" size="1.778" layer="95" xref="yes"/>
-</segment>
-<segment>
 <pinref part="D27" gate="G$1" pin="C"/>
 <pinref part="GND11" gate="1" pin="GND"/>
@@
 <pinref part="GND17" gate="1" pin="GND"/>
 </segment>
-</net>
-<net name="3.3V" class="0">
-<segment>
-<pinref part="SUPPLY5" gate="G$1" pin="3.3V"/>
-<wire x1="-73.66" y1="30.48" x2="-73.66" y2="27.94" width="0.1524" layer="91"/>
-<wire x1="-73.66" y1="27.94" x2="-68.58" y2="27.94" width="0.1524" layer="91"/>
-<wire x1="-88.9" y1="27.94" x2="-83.82" y2="27.94" width="0.1524" layer="91"/>
-<junction x="-73.66" y="27.94"/>
-<pinref part="C34" gate="G$1" pin="1"/>
-<pinref part="C35" gate="G$1" pin="1"/>
-<wire x1="-83.82" y1="27.94" x2="-73.66" y2="27.94" width="0.1524" layer="91"/>
-<junction x="-83.82" y="27.94"/>
-<pinref part="U1" gate="G$1" pin="VCC"/>
-</segment>
-<segment>
-<pinref part="SUPPLY17" gate="G$1" pin="3.3V"/>
-<wire x1="-139.7" y1="-35.56" x2="-139.7" y2="-38.1" width="0.1524" layer="91"/>
-<pinref part="R5" gate="G$1" pin="1"/>
-<wire x1="-144.78" y1="-40.64" x2="-144.78" y2="-38.1" width="0.1524" layer="91"/>
-<wire x1="-144.78" y1="-38.1" x2="-139.7" y2="-38.1" width="0.1524" layer="91"/>
-<pinref part="SP1" gate="S1" pin="+"/>
-<wire x1="-139.7" y1="-38.1" x2="-139.7" y2="-40.64" width="0.1524" layer="91"/>
-<junction x="-139.7" y="-38.1"/>
-</segment>
-<segment>
-<pinref part="R20" gate="G$1" pin="1"/>
+<segment>
+<pinref part="GND37" gate="1" pin="GND"/>
+<pinref part="D33" gate="G$1" pin="GND"/>
+<wire x1="-27.94" y1="-63.5" x2="-35.56" y2="-63.5" width="0.1524" layer="91"/>
+</segment>
+<segment>
 <pinref part="C6" gate="G$1" pin="1"/>
-<pinref part="D33" gate="G$1" pin="VS"/>
-<wire x1="-35.56" y1="-53.34" x2="-30.48" y2="-53.34" width="0.1524" layer="91"/>
-<junction x="-30.48" y="-53.34"/>
-</segment>
-<segment>
-<pinref part="R20" gate="G$1" pin="2"/>
-<wire x1="-20.32" y1="-53.34" x2="-17.78" y2="-53.34" width="0.1524" layer="91"/>
-<wire x1="-15.24" y1="-53.34" x2="-17.78" y2="-53.34" width="0.1524" layer="91"/>
-<label x="-15.24" y="-53.34" size="1.778" layer="95" xref="yes"/>
+<pinref part="GND41" gate="1" pin="GND"/>
 </segment>
 </net>
@@
 <wire x1="-172.72" y1="-10.16" x2="-175.26" y2="-10.16" width="0.1524" layer="91"/>
 <label x="-175.26" y="-10.16" size="1.27" layer="95" rot="R180" xref="yes"/>
+</segment>
+</net>
+<net name="3.3V" class="0">
+<segment>
+<pinref part="R20" gate="G$1" pin="2"/>
+<wire x1="-20.32" y1="-53.34" x2="-15.24" y2="-53.34" width="0.1524" layer="91"/>
+<label x="-15.24" y="-53.34" size="1.778" layer="95" xref="yes"/>
+</segment>
+<segment>
+<pinref part="SUPPLY17" gate="G$1" pin="3.3V"/>
+<pinref part="SP1" gate="S1" pin="+"/>
+<wire x1="-139.7" y1="-35.56" x2="-139.7" y2="-38.1" width="0.1524" layer="91"/>
+<pinref part="R5" gate="G$1" pin="1"/>
+<wire x1="-139.7" y1="-38.1" x2="-139.7" y2="-40.64" width="0.1524" layer="91"/>
+<wire x1="-144.78" y1="-40.64" x2="-144.78" y2="-38.1" width="0.1524" layer="91"/>
+<wire x1="-144.78" y1="-38.1" x2="-139.7" y2="-38.1" width="0.1524" layer="91"/>
+<junction x="-139.7" y="-38.1"/>
+</segment>
+<segment>
+<pinref part="SUPPLY5" gate="G$1" pin="3.3V"/>
+<wire x1="-73.66" y1="30.48" x2="-73.66" y2="27.94" width="0.1524" layer="91"/>
+<wire x1="-73.66" y1="27.94" x2="-68.58" y2="27.94" width="0.1524" layer="91"/>
+<wire x1="-88.9" y1="27.94" x2="-83.82" y2="27.94" width="0.1524" layer="91"/>
+<junction x="-73.66" y="27.94"/>
+<pinref part="C34" gate="G$1" pin="1"/>
+<pinref part="C35" gate="G$1" pin="1"/>
+<wire x1="-83.82" y1="27.94" x2="-73.66" y2="27.94" width="0.1524" layer="91"/>
+<junction x="-83.82" y="27.94"/>
+<pinref part="U1" gate="G$1" pin="VCC"/>
+</segment>
+<segment>
+<pinref part="R20" gate="G$1" pin="1"/>
+<pinref part="D33" gate="G$1" pin="VS"/>
+<wire x1="-30.48" y1="-53.34" x2="-35.56" y2="-53.34" width="0.1524" layer="91"/>
+<wire x1="-30.48" y1="-53.34" x2="-30.48" y2="-50.8" width="0.1524" layer="91"/>
+<junction x="-30.48" y="-53.34"/>
+<pinref part="C6" gate="G$1" pin="2"/>
 </segment>
 </net>
@@
 <attribute name="VALUE" x="-106.68" y="35.56" size="1.27" layer="96" align="top-left"/>
 </instance>
+<instance part="TP2" gate="G$1" x="129.54" y="73.66" smashed="yes">
+<attribute name="NAME" x="128.27" y="74.93" size="1.778" layer="95"/>
+<attribute name="TP_SIGNAL_NAME" x="130.81" y="72.39" size="1.778" layer="97"/>
+</instance>
+<instance part="TP3" gate="G$1" x="-88.9" y="12.7" smashed="yes">
+<attribute name="NAME" x="-90.17" y="13.97" size="1.778" layer="95"/>
+<attribute name="TP_SIGNAL_NAME" x="-87.63" y="11.43" size="1.778" layer="97"/>
+</instance>
 </instances>
 <busses>
@@
 <pinref part="U2" gate="G$1" pin="VDD3P3_CPU"/>
 <pinref part="U2" gate="G$1" pin="VDDA"/>
+<label x="20.32" y="83.82" size="1.778" layer="95" xref="yes"/>
 </segment>
 <segment>
@@
 </segment>
 </net>
-<net name="T_B" class="0">
-<segment>
-<wire x1="127" y1="71.12" x2="129.54" y2="71.12" width="0.1524" layer="91"/>
-<label x="129.54" y="71.12" size="1.27" layer="95" xref="yes"/>
-<pinref part="U2" gate="G$1" pin="(ADC2:1/TOUCH1/RTC11/CLK_OUT1)GPIO0"/>
-</segment>
+<net name="T_B2" class="0">
 <segment>
 <pinref part="Q4" gate="Q2" pin="C"/>
@@
 <wire x1="-88.9" y1="10.16" x2="-91.44" y2="10.16" width="0.1524" layer="91"/>
 <label x="-91.44" y="10.16" size="1.27" layer="95" rot="R180" xref="yes"/>
+<pinref part="TP3" gate="G$1" pin="PP"/>
+<junction x="-88.9" y="10.16"/>
 </segment>
 </net>
@@
 </segment>
 </net>
+<net name="T_B1" class="0">
+<segment>
+<pinref part="U2" gate="G$1" pin="(ADC2:1/TOUCH1/RTC11/CLK_OUT1)GPIO0"/>
+<pinref part="TP2" gate="G$1" pin="PP"/>
+<wire x1="127" y1="71.12" x2="129.54" y2="71.12" width="0.1524" layer="91"/>
+<label x="129.54" y="71.12" size="1.778" layer="95" xref="yes"/>
+</segment>
+</net>
