File: Hardware/Release/tc0xC_prod.sch (EAGLE design)
At the start: 102 parts, among them IC1 AP2112M-3.3TRG1, Q1 2.5A/30V, Q2 MBT3904DW1T1, Q3 600mA/40V, Q4 MBT3904DW1T1, U2 ESP3212, U4 FT231XS, U5 W25Q32FVSS, Y1 26MHz, Y2 32.768kHz

Commit message: add silk. update layout to fit plastics. minor adjustments to layout.
Connections:
- new net N$17: C6.2, D33.VS, R20.1
- net 3.3V: no longer C6.2, D33.VS, R20.1
Changed lines of the file:
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@@
 <?xml version="1.0" encoding="utf-8"?>
 <!DOCTYPE eagle SYSTEM "eagle.dtd">
-<eagle version="9.3.0">
+<eagle version="9.6.2">
 <drawing>
 <settings>
@@
 <setting verticaltext="up"/>
 </settings>
-<grid distance="0.1" unitdist="inch" unit="inch" style="lines" multiple="1" display="no" altdistance="0.01" altunitdist="inch" altunit="inch"/>
+<grid distance="0.1" unitdist="inch" unit="inch" style="lines" multiple="1" display="yes" altdistance="0.01" altunitdist="inch" altunit="inch"/>
 <layers>
 <layer number="1" name="Top" color="4" fill="1" visible="no" active="no"/>
@@
 <part name="GND16" library="SparkFun-Aesthetics" deviceset="GND" device=""/>
 <part name="SUPPLY23" library="SparkFun-Aesthetics" deviceset="3.3V" device=""/>
-<part name="S2" library="IDEO-Switches" deviceset="CUS-12B" device=""/>
+<part name="S2" library="IDEO-Switches" deviceset="CUS-12B" device="" override_package3d_urn="urn:adsk.eagle:package:39905697/2" override_package_urn="urn:adsk.eagle:footprint:39905698/1"/>
 <part name="SUPPLY15" library="SparkFun-Aesthetics" deviceset="V_BATT" device=""/>
 <part name="GND34" library="SparkFun-Aesthetics" deviceset="GND" device=""/>
-<part name="J1" library="SparkFun-Connectors-new" deviceset="USB_MICRO-B" device=""/>
+<part name="J1" library="SparkFun-Connectors-new" deviceset="USB_MICRO-B" device="" override_package3d_urn="urn:adsk.eagle:package:39905683/2" override_package_urn="urn:adsk.eagle:footprint:39905684/1"/>
 <part name="GND39" library="SparkFun-Aesthetics" deviceset="GND" device=""/>
 <part name="IC1" library="AP2112M-3.3TRG1" deviceset="AP2112M-3.3TRG1" device=""/>
@@
 <part name="U$3" library="microbuilder" deviceset="GND" device=""/>
 <part name="D33" library="TSOP36256" deviceset="TSOP36256" device="TT"/>
-<part name="D27" library="VSMB2020X01" deviceset="VSMB2020X01" device=""/>
-<part name="D28" library="VSMB2020X01" deviceset="VSMB2020X01" device=""/>
+<part name="D27" library="VSMB2020X01" deviceset="VSMB2020X01" device="" override_package3d_urn="urn:adsk.eagle:package:39905680/2" override_package_urn="urn:adsk.eagle:footprint:39905681/1"/>
+<part name="D28" library="VSMB2020X01" deviceset="VSMB2020X01" device="" override_package3d_urn="urn:adsk.eagle:package:39905717/2" override_package_urn="urn:adsk.eagle:footprint:39905718/1"/>
 <part name="R19" library="SparkFun-Resistors" deviceset="10KOHM" device="-0603-1/10W-1%" value="10k"/>
 <part name="SUPPLY3" library="SparkFun-Aesthetics" deviceset="3.3V" device=""/>
@@
 <part name="R21" library="SparkFun-Resistors" deviceset="10KOHM" device="-0603-1/10W-1%" value="8.2"/>
 <part name="R22" library="SparkFun-Resistors" deviceset="10KOHM" device="-0603-1/10W-1%" value="8.2"/>
-<part name="S3" library="TL3340AF160QG" deviceset="TL3340AF160QG" device=""/>
+<part name="S3" library="TL3340AF160QG" deviceset="TL3340AF160QG" device="" override_package3d_urn="urn:adsk.eagle:package:39905701/2" override_package_urn="urn:adsk.eagle:footprint:39905702/1"/>
 <part name="TP2" library="testpad" library_urn="urn:adsk.eagle:library:385" deviceset="TPS" device="TP08R" package3d_urn="urn:adsk.eagle:package:27956/1"/>
 <part name="TP3" library="testpad" library_urn="urn:adsk.eagle:library:385" deviceset="TPS" device="TP08R" package3d_urn="urn:adsk.eagle:package:27956/1"/>
@@
 <pinref part="U1" gate="G$1" pin="VCC"/>
 </segment>
-<segment>
+</net>
+<net name="N$17" class="0">
+<segment>
+<pinref part="C6" gate="G$1" pin="2"/>
 <pinref part="R20" gate="G$1" pin="1"/>
+<wire x1="-30.48" y1="-50.8" x2="-30.48" y2="-53.34" width="0.1524" layer="91"/>
 <pinref part="D33" gate="G$1" pin="VS"/>
 <wire x1="-30.48" y1="-53.34" x2="-35.56" y2="-53.34" width="0.1524" layer="91"/>
-<wire x1="-30.48" y1="-53.34" x2="-30.48" y2="-50.8" width="0.1524" layer="91"/>
 <junction x="-30.48" y="-53.34"/>
-<pinref part="C6" gate="G$1" pin="2"/>
 </segment>
 </net>
@@
 packages will not be understood (or retained) with this version.
 </note>
+<note version="9.4" severity="warning">
+Since Version 9.4, EAGLE supports the overriding of 3D packages
+in schematics and board files. Those overridden 3d packages
+will not be understood (or retained) with this version.
+</note>
 </compatibility>

Commit message: Review CAMS, Art, Schematic Updates - Pre final route
Parts:
- added D29, D30: VSMB2020X01, VSMB2020X01:VSMB2020X01
- added R23, R24: 8.2, SparkFun-Resistors:10KOHM-0603-1/10W-1%
- added U$1, U$4: T2N7002BK, T2N7002BK:T2N7002BK
Connections:
- new net N$19: D29.C, U$1.D
- new net N$20: D30.C, U$4.D
- new net N$21: D29.A, R23.2
- new net N$22: D30.A, R24.2
- net 3.3V: now also R23.1, R24.1
- net GND: now also U$1.S, U$4.S
- net IR_OUT: now also U$1.G, U$4.G
Changed lines of the file:
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@@
 <setting verticaltext="up"/>
 </settings>
-<grid distance="0.1" unitdist="inch" unit="inch" style="lines" multiple="1" display="yes" altdistance="0.01" altunitdist="inch" altunit="inch"/>
+<grid distance="0.1" unitdist="inch" unit="inch" style="lines" multiple="1" display="no" altdistance="0.01" altunitdist="inch" altunit="inch"/>
 <layers>
 <layer number="1" name="Top" color="4" fill="1" visible="no" active="no"/>
@@
 <part name="C6" library="SparkFun-Capacitors" deviceset="10PF" device="-0603-50V-5%" value="0.1uF"/>
 <part name="GND41" library="supply1" library_urn="urn:adsk.eagle:library:371" deviceset="GND" device=""/>
+<part name="D29" library="VSMB2020X01" deviceset="VSMB2020X01" device="" override_package3d_urn="urn:adsk.eagle:package:39905680/2" override_package_urn="urn:adsk.eagle:footprint:39905681/1"/>
+<part name="D30" library="VSMB2020X01" deviceset="VSMB2020X01" device="" override_package3d_urn="urn:adsk.eagle:package:39905680/2" override_package_urn="urn:adsk.eagle:footprint:39905681/1"/>
+<part name="U$1" library="T2N7002BK" deviceset="T2N7002BK" device=""/>
+<part name="U$4" library="T2N7002BK" deviceset="T2N7002BK" device=""/>
+<part name="GND42" library="SparkFun-Aesthetics" deviceset="GND" device=""/>
+<part name="GND43" library="SparkFun-Aesthetics" deviceset="GND" device=""/>
+<part name="SUPPLY4" library="SparkFun-Aesthetics" deviceset="3.3V" device=""/>
+<part name="SUPPLY6" library="SparkFun-Aesthetics" deviceset="3.3V" device=""/>
+<part name="R23" library="SparkFun-Resistors" deviceset="10KOHM" device="-0603-1/10W-1%" value="8.2"/>
+<part name="R24" library="SparkFun-Resistors" deviceset="10KOHM" device="-0603-1/10W-1%" value="8.2"/>
 </parts>
 <sheets>
@@
 <attribute name="VALUE" x="-27.94" y="-38.1" size="1.778" layer="96" rot="R180"/>
 </instance>
+<instance part="D29" gate="G$1" x="-160.02" y="63.5" smashed="yes" rot="R270">
+<attribute name="NAME" x="-155.194" y="67.056" size="1.27" layer="95" rot="R270"/>
+<attribute name="VALUE" x="-163.322" y="67.056" size="1.27" layer="96" rot="R270"/>
+</instance>
+<instance part="D30" gate="G$1" x="-109.22" y="63.5" smashed="yes" rot="R270">
+<attribute name="NAME" x="-104.394" y="67.056" size="1.27" layer="95" rot="R270"/>
+<attribute name="VALUE" x="-112.522" y="67.056" size="1.27" layer="96" rot="R270"/>
+</instance>
+<instance part="U$1" gate="G$1" x="-162.56" y="48.26" smashed="yes">
+<attribute name="NAME" x="-156.21" y="49.53" size="1.778" layer="95"/>
+<attribute name="VALUE" x="-156.21" y="46.99" size="1.778" layer="96"/>
+</instance>
+<instance part="U$4" gate="G$1" x="-111.76" y="48.26" smashed="yes">
+<attribute name="NAME" x="-105.41" y="49.53" size="1.778" layer="95"/>
+<attribute name="VALUE" x="-105.41" y="46.99" size="1.778" layer="96"/>
+</instance>
+<instance part="GND42" gate="1" x="-160.02" y="35.56" smashed="yes" rot="MR0">
+<attribute name="VALUE" x="-157.48" y="33.02" size="1.778" layer="96" rot="MR0"/>
+</instance>
+<instance part="GND43" gate="1" x="-109.22" y="35.56" smashed="yes" rot="MR0">
+<attribute name="VALUE" x="-106.68" y="33.02" size="1.778" layer="96" rot="MR0"/>
+</instance>
+<instance part="SUPPLY4" gate="G$1" x="-160.02" y="86.36" smashed="yes">
+<attribute name="VALUE" x="-161.036" y="89.916" size="1.778" layer="96"/>
+</instance>
+<instance part="SUPPLY6" gate="G$1" x="-109.22" y="86.36" smashed="yes">
+<attribute name="VALUE" x="-110.236" y="89.916" size="1.778" layer="96"/>
+</instance>
+<instance part="R23" gate="G$1" x="-160.02" y="78.74" smashed="yes" rot="R270">
+<attribute name="NAME" x="-158.496" y="78.74" size="1.778" layer="95" font="vector" rot="R270" align="bottom-center"/>
+<attribute name="VALUE" x="-161.544" y="78.74" size="1.778" layer="96" font="vector" rot="R270" align="top-center"/>
+</instance>
+<instance part="R24" gate="G$1" x="-109.22" y="78.74" smashed="yes" rot="R270">
+<attribute name="NAME" x="-107.696" y="78.74" size="1.778" layer="95" font="vector" rot="R270" align="bottom-center"/>
+<attribute name="VALUE" x="-110.744" y="78.74" size="1.778" layer="96" font="vector" rot="R270" align="top-center"/>
+</instance>
 </instances>
 <busses>
@@
 <pinref part="C6" gate="G$1" pin="1"/>
 <pinref part="GND41" gate="1" pin="GND"/>
+</segment>
+<segment>
+<pinref part="U$1" gate="G$1" pin="S"/>
+<pinref part="GND42" gate="1" pin="GND"/>
+<wire x1="-160.02" y1="40.64" x2="-160.02" y2="38.1" width="0.1524" layer="91"/>
+</segment>
+<segment>
+<pinref part="U$4" gate="G$1" pin="S"/>
+<pinref part="GND43" gate="1" pin="GND"/>
+<wire x1="-109.22" y1="40.64" x2="-109.22" y2="38.1" width="0.1524" layer="91"/>
 </segment>
 </net>
@@
 <label x="-68.58" y="-33.02" size="1.778" layer="95" rot="R180" xref="yes"/>
 </segment>
+<segment>
+<pinref part="U$1" gate="G$1" pin="G"/>
+<wire x1="-170.18" y1="45.72" x2="-177.8" y2="45.72" width="0.1524" layer="91"/>
+<label x="-177.8" y="45.72" size="1.778" layer="95" rot="R180" xref="yes"/>
+</segment>
+<segment>
+<pinref part="U$4" gate="G$1" pin="G"/>
+<wire x1="-119.38" y1="45.72" x2="-127" y2="45.72" width="0.1524" layer="91"/>
+<label x="-127" y="45.72" size="1.778" layer="95" rot="R180" xref="yes"/>
+</segment>
 </net>
 <net name="FLASH_SCS" class="0">
@@
 <pinref part="U1" gate="G$1" pin="VCC"/>
 </segment>
+<segment>
+<pinref part="SUPPLY4" gate="G$1" pin="3.3V"/>
+<pinref part="R23" gate="G$1" pin="1"/>
+<wire x1="-160.02" y1="86.36" x2="-160.02" y2="83.82" width="0.1524" layer="91"/>
+</segment>
+<segment>
+<pinref part="SUPPLY6" gate="G$1" pin="3.3V"/>
+<pinref part="R24" gate="G$1" pin="1"/>
+<wire x1="-109.22" y1="86.36" x2="-109.22" y2="83.82" width="0.1524" layer="91"/>
+</segment>
 </net>
 <net name="N$17" class="0">
@@
 </segment>
 </net>
+<net name="N$19" class="0">
+<segment>
+<pinref part="D29" gate="G$1" pin="C"/>
+<pinref part="U$1" gate="G$1" pin="D"/>
+<wire x1="-160.02" y1="58.42" x2="-160.02" y2="53.34" width="0.1524" layer="91"/>
+</segment>
+</net>
+<net name="N$20" class="0">
+<segment>
+<pinref part="D30" gate="G$1" pin="C"/>
+<pinref part="U$4" gate="G$1" pin="D"/>
+<wire x1="-109.22" y1="58.42" x2="-109.22" y2="53.34" width="0.1524" layer="91"/>
+</segment>
+</net>
+<net name="N$21" class="0">
+<segment>
+<pinref part="R23" gate="G$1" pin="2"/>
+<pinref part="D29" gate="G$1" pin="A"/>
+<wire x1="-160.02" y1="73.66" x2="-160.02" y2="71.12" width="0.1524" layer="91"/>
+</segment>
+</net>
+<net name="N$22" class="0">
+<segment>
+<pinref part="R24" gate="G$1" pin="2"/>
+<pinref part="D30" gate="G$1" pin="A"/>
+<wire x1="-109.22" y1="73.66" x2="-109.22" y2="71.12" width="0.1524" layer="91"/>
+</segment>
+</net>

Commit message: Hardware and Art dirs
Parts:
- removed D29, D30: VSMB2020X01, VSMB2020X01:VSMB2020X01
- removed TP2, TP3: TPSTP08R, testpad:TPSTP08R
- removed U$1, U$4: T2N7002BK, T2N7002BK:T2N7002BK
- added Q5, Q6: MOSFET-NCH-RUC002N05HZGT116, Rob-DiscreteSemi:MOSFET-NCH-RUC002N05HZGT116
- added R25: 100K, SparkFun-Resistors:10KOHM-0603-1/10W-1%
- added R26: 22, SparkFun-Resistors:10KOHM-0603-1/10W-1%
- R22: value 8.2 -> 240
- R23: value 8.2 -> 22
- R24: value 8.2 -> 100K
- renumbered C75 to C7FIVE
Connections:
- removed net T_B1: TP2.PP, U2.(ADC2:1/TOUCH1/RTC11/CLK_OUT1)GPIO0
- removed net T_B2: Q4Q2.C, TP3.PP
- new net GPIO-0: Q4Q2.C, U2.(ADC2:1/TOUCH1/RTC11/CLK_OUT1)GPIO0
- net 3.3V: now also R26.1; no longer R24.1
- net GND: now also Q5.S, Q6.S, R24.2, R25.2; no longer D27.C, D28.C, U$1.S, U$4.S
- net IR_OUT: no longer U$1.G, U$4.G
- net N$19: now also D28.C, Q5.D; no longer D29.C, U$1.D
- net N$20: now also D28.A, R23.2; no longer D30.C, U$4.D
- net N$21: now also D27.C, Q6.D; no longer D29.A, R23.2
- net N$22: now also D27.A, R26.2; no longer D30.A, R24.2
- net N$5: now also Q6.G, R25.1; no longer D27.A
- net N$6: now also Q5.G, R24.1; no longer D28.A
Other:
- moved on the sheet: D27, D28, R21, R22, R23, R24
